File: ADC.kicad_pcb (KiCad board)
At the start: 2 copper layers, 195 parts, among them J1 Conn_01x03_Pin, J2 Screw_Terminal_01x02, J3 Screw_Terminal_01x09, SW1 SW_SPDT, U1 ADS1256IDBR, U10 CD4514BM, U11 ADG5412FBCPZ-RL7, U12 ADR421ARMZ, U13 OPA211ID, U14 ADG5412FBCPZ-RL7, U15 OPA211ID, U16 ADG5412FBCPZ-RL7, U17 OPA211ID, U18 CD4072BM, U19 CD4514BM, U2 MCU-STM32F407VET6_LQFP100_, U20 ADG5412FBCPZ-RL7, U21 ADG5412FBCPZ-RL7, U22 ADG5412FBCPZ-RL7, U23 ADG5412FBCPZ-RL7, U24 OPA211ID, U25 OPA211ID, U26 OPA211ID, U27 OPA211ID, U28 CD4043BPWR, U29 TLV1704AIPWR, U3 ADM2483xRW, U30 TLV1704AIPWR, U31 TLV1704AIPWR, U32 CD4072BM, U4 LM2596S-5, U5 DCP010505BP, U6 TLV1704AIPWR, U7 OPA211ID, U8 AMS1117-3.3, U9 ADG5412FBCPZ-RL7, Y1 8MHz, Y2 ABM3B-25.000MHZ-D2Y-T

Commit message: chia khu linh kiện PCB
Parts:
- moved J1 996.0 mm to (1102.6, 83.1)
- moved RV1 996.0 mm to (1102.0, 76.7)
- moved R18 987.0 mm to (1105.0, 51.5)
- moved R19 987.0 mm to (1105.0, 53.5)
- moved R20 987.0 mm to (1105.0, 55.5)
- moved R21 987.0 mm to (1105.0, 57.5)
- moved R22 987.0 mm to (1105.0, 59.5)
- moved R24 987.0 mm to (1105.0, 63.4)
- moved D16 979.8 mm to (1118.6, 79.0)
- moved D6 979.8 mm to (1118.6, 71.5)
- moved U3 966.5 mm to (1134.1, 76.0)
- moved C39 966.5 mm to (1144.8, 93.8)
- moved C40 966.5 mm to (1148.8, 83.7)
- moved C38 949.7 mm to (1130.5, 58.5)
- moved C41 949.7 mm to (1130.5, 60.4)
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Connections:
- D10 pad 1: VinP3 -> VinN2
- D11 pad 1: VinN3 -> VinP2
- D12 pad 1: VinP4 -> VinN1
- D13 pad 1: VinN4 -> VinP1
- D14 pad 1: VinP1 -> VinP4
- D14 pad 2: VinN1 -> VinN4
- D15 pad 1: VinP1 -> VinN4
- D19 pad 1: VinP2 -> VinP3
- D19 pad 2: VinN2 -> VinN3
- D21 pad 1: VinP3 -> VinP2
- D21 pad 2: VinN3 -> VinN2
- D23 pad 1: VinP4 -> VinP1
- D23 pad 2: VinN4 -> VinN1
- D7 pad 1: VinN1 -> VinP4
- D8 pad 1: VinP2 -> VinN3
- D9 pad 1: VinN2 -> VinP3
- J3 pad 1: VinP1 -> GND
- J3 pad 2: VinN1 -> VinP1
- J3 pad 3: VinP2 -> VinN1
- J3 pad 4: VinN2 -> VinP2
- J3 pad 5: VinP3 -> VinN2
- J3 pad 6: VinN3 -> VinP3
- J3 pad 7: VinP4 -> VinN3
- J3 pad 8: VinN4 -> VinP4
- J3 pad 9: GND -> VinN4
- U13 pad 3: VinP2 -> VinN1
- U15 pad 3: VinP3 -> VinP2
- U17 pad 3: VinP4 -> VinN2
- U2 pad 15: RESET -> unconnected-(U2-PC0-Pad15)
- U2 pad 17: DECODER1_1 -> unconnected-(U2-PC2-Pad17)
- U2 pad 18: DECODER1_2 -> unconnected-(U2-PC3-Pad18)
- U2 pad 33: DECODER1_3 -> unconnected-(U2-PC4-Pad33)
- U2 pad 34: DECODER1_4 -> unconnected-(U2-PC5-Pad34)
- U2 pad 57: unconnected-(U2-PD10-Pad57) -> DECODER1_1
- U2 pad 58: unconnected-(U2-PD11-Pad58) -> DECODER1_2
- U2 pad 59: unconnected-(U2-PD12-Pad59) -> DECODER1_3
- U2 pad 60: unconnected-(U2-PD13-Pad60) -> DECODER1_4
- U2 pad 62: unconnected-(U2-PD15-Pad62) -> RESET
- U2 pad 63: unconnected-(U2-PC6-Pad63) -> DECODER2_1
- U2 pad 64: DECODER2_1 -> DECODER2_2
- U2 pad 65: DECODER2_2 -> DECODER2_3
- U2 pad 66: DECODER2_3 -> DECODER2_4
- U2 pad 78: DECODER2_4 -> unconnected-(U2-PC10-Pad78)
- U24 pad 3: VinP7 -> VinP4
- U25 pad 3: VinP8 -> VinN4
- U26 pad 3: VinP5 -> VinP3
- U27 pad 3: VinP6 -> VinN3

Commit message: update
Parts:
- C7, D1, D10, D11, D12, D13, D14, D15, D17, D19, D2, D21, D23, D3, D7, D8, D9, F1, L1, L2, R1, R2, R25, R26, R27, R28, R29, R3, R30, R31, R32, R33, R34, R35, R36, R37, R38, R39, R40, R41, R42, R43, R44, R45, R46, R47, R48, R49, R50, R51, R52, R53, R54, R55, R56, R57, R58, R59, R60, R61, R62, R63, R64, R65, R66, R67, R68, R69, R70, U11, U13, U14, U15, U16, U17, U20, U21, U22, U23, U24, U25, U26, U27, U4, U7, U8, U9: moved to B.Cu
- moved U28 289.2 mm to (437.3, 478.1), turned to -90 degrees
- moved R71 232.5 mm to (333.0, 452.0)
- moved R72 232.5 mm to (333.0, 454.0)
- moved R73 232.5 mm to (333.0, 456.0)
- moved R74 232.5 mm to (333.0, 458.0)
- moved R75 232.5 mm to (350.0, 488.2)
- moved R76 232.5 mm to (350.0, 489.7)
- moved R77 232.5 mm to (350.0, 491.7)
- moved R78 232.5 mm to (350.0, 493.7)
- moved R79 232.5 mm to (331.5, 465.8)
- moved R80 232.5 mm to (331.5, 467.8)
- moved R81 232.5 mm to (331.5, 469.8)
- moved R82 232.5 mm to (331.5, 471.8)
- moved R83 232.5 mm to (332.2, 501.3)
- moved R84 232.5 mm to (331.2, 524.2)
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Routing:
- net GND: track 0.00 -> 137.1 mm
- net VinP1: track 0.00 -> 51.0 mm
- net +5V: track 0.00 -> 42.8 mm
- net VinN1: track 0.00 -> 34.8 mm
- net VinN4: track 0.00 -> 31.7 mm
- net VinP4: track 0.00 -> 29.8 mm
- net VinP2: track 0.00 -> 27.8 mm
- net VinN2: track 0.00 -> 23.6 mm
- net VinN3: track 0.00 -> 23.5 mm
- net VinP3: track 0.00 -> 21.8 mm
- net +3.3V: track 0.00 -> 16.1 mm
- net Net-(PS1-+VIN): track 0.00 -> 15.3 mm
- net Net-(D1-K): track 0.00 -> 15.1 mm
- net +12V_IN: track 0.00 -> 6.98 mm
- net +12V: track 0.00 -> 3.55 mm
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
Commit message: xong bộ bám điện áp, khuếch đại
Parts:
- moved R64 125.7 mm to (450.5, 679.6)
- moved R63 123.7 mm to (448.5, 679.6)
- moved R62 121.7 mm to (446.5, 679.6)
- moved U25 121.4 mm to (440.5, 683.1), turned to 0 degrees
- moved R52 120.7 mm to (446.8, 686.6), turned to 0 degrees
- moved R48 112.7 mm to (450.3, 686.6), turned to 0 degrees
- moved R61 111.1 mm to (451.5, 650.2)
- moved U21 110.9 mm to (448.5, 683.4)
- moved U24 109.9 mm to (441.5, 653.9), turned to 0 degrees
- moved R60 109.0 mm to (449.5, 650.2)
- moved R59 107.0 mm to (447.5, 650.2)
- moved R56 106.9 mm to (443.2, 686.6), turned to 0 degrees
- moved R47 102.0 mm to (451.3, 657.2), turned to 0 degrees
- moved R51 98.8 mm to (447.8, 657.2), turned to 0 degrees
- moved U20 97.0 mm to (449.5, 654.0)
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Routing:
- net +12V: track 3.55 -> 61.3 mm, vias 0 -> 8
- net GND: track 137.1 -> 177.8 mm
- net VinP1: track 51.0 -> 65.4 mm
- net Net-(U25--IN): track 0.00 -> 13.6 mm
- net Net-(U24--IN): track 0.00 -> 13.5 mm
- net Net-(U7--IN): track 0.00 -> 13.5 mm
- net Net-(U26--IN): track 0.00 -> 13.5 mm
- net Net-(U15--IN): track 0.00 -> 13.4 mm
- net Net-(U27--IN): track 0.00 -> 13.3 mm
- net Net-(U17--IN): track 0.00 -> 13.3 mm
- net Net-(U13--IN): track 0.00 -> 13.2 mm
- net ADC1: track 0.00 -> 12.9 mm, vias 0 -> 2
- net Net-(U17-OUT): track 0.00 -> 12.1 mm
- net Net-(U26-OUT): track 0.00 -> 11.8 mm
- net Net-(U25-OUT): track 0.00 -> 11.7 mm
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
Commit message: đã tìm được đường đi cho nhưng dây phức tạp
Parts:
- moved C9 326.4 mm to (768.1, 254.5)
- moved D4 326.4 mm to (841.6, 233.7)
- moved D5 326.4 mm to (841.6, 237.3)
- moved R18 326.4 mm to (834.1, 233.7)
- moved R19 326.4 mm to (834.1, 235.7)
- moved R20 326.4 mm to (834.1, 237.7)
- moved R21 326.4 mm to (834.1, 239.7)
- moved R22 326.4 mm to (834.1, 241.7)
- moved R24 326.4 mm to (834.1, 245.7)
- moved U5 326.4 mm to (782.4, 251.7)
- moved C10 326.4 mm to (752.6, 246.5)
- moved C11 326.4 mm to (752.6, 249.5)
- moved C38 326.4 mm to (859.7, 240.7)
- moved C39 326.4 mm to (874.0, 276.0)
- moved C40 326.4 mm to (878.0, 266.0)
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Routing:
- net ADC8: track 6.78 -> 557.0 mm, vias 2 -> 3
- net ADC1: track 12.9 -> 509.5 mm, vias 2 -> 3
- net ADC7: track 6.11 -> 487.9 mm, vias 2 -> 3
- net ADC2: track 6.65 -> 462.4 mm, vias 2 -> 3
- net ADC6: track 5.79 -> 447.9 mm, vias 2 -> 3
- net ADC3: track 5.75 -> 427.6 mm, vias 2 -> 3
- net ADC5: track 6.36 -> 415.0 mm, vias 2 -> 3
- net ADC4: track 5.89 -> 412.4 mm, vias 2 -> 3
- net VinN4: track 34.3 -> 194.3 mm
- net VinN1: track 37.8 -> 188.5 mm
- net VinP4: track 32.6 -> 181.9 mm
- net VinP1: track 65.4 -> 214.3 mm
- net VinP2: track 30.7 -> 179.3 mm
- net VinN2: track 26.5 -> 170.6 mm
- net VinN3: track 27.6 -> 171.5 mm
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
Commit message: update
Parts:
- moved U10 85.0 mm to (472.1, 410.9), turned to -90 degrees
- moved U19 84.4 mm to (474.1, 499.6)
Connections:
- U10 pad 10: Net-(U10-S1) -> /2_IN4
- U10 pad 11: Net-(U10-S0) -> /2_in3
- U10 pad 13: Net-(U10-S13) -> /3_IN2
- U10 pad 14: Net-(U10-S12) -> /3_IN1
- U10 pad 15: Net-(U10-S15) -> /3_IN4
- U10 pad 16: Net-(U10-S14) -> /3_IN3
- U10 pad 17: Net-(U10-S9) -> /4_IN2
- U10 pad 18: Net-(U10-S8) -> /4_IN1
- U10 pad 19: Net-(U10-S11) -> /4_IN4
- U10 pad 20: Net-(U10-S10) -> /4_IN3
- U10 pad 4: Net-(U10-S7) -> /1_IN2
- U10 pad 5: Net-(U10-S6) -> /1_IN1
- U10 pad 6: Net-(U10-S5) -> /1_IN4
- U10 pad 7: Net-(U10-S4) -> /1_IN3
- U10 pad 8: Net-(U10-S3) -> /2_IN2
- U10 pad 9: Net-(U10-S2) -> /2_IN1
- U11 pad 14: Net-(U10-S5) -> /2_IN2
- U11 pad 15: Net-(U10-S4) -> /2_IN1
- U11 pad 6: Net-(U10-S7) -> /2_IN4
- U11 pad 7: Net-(U10-S6) -> /2_in3
- U14 pad 14: Net-(U10-S9) -> /3_IN2
- U14 pad 15: Net-(U10-S8) -> /3_IN1
- U14 pad 6: Net-(U10-S11) -> /3_IN4
- U14 pad 7: Net-(U10-S10) -> /3_IN3
- U16 pad 14: Net-(U10-S13) -> /4_IN2
- U16 pad 15: Net-(U10-S12) -> /4_IN1
- U16 pad 6: Net-(U10-S15) -> /4_IN4
- U16 pad 7: Net-(U10-S14) -> /4_IN3
- U9 pad 14: Net-(U10-S1) -> /1_IN2
- U9 pad 15: Net-(U10-S0) -> /1_IN1
- U9 pad 6: Net-(U10-S3) -> /1_IN4
- U9 pad 7: Net-(U10-S2) -> /1_IN3
Routing:
- net DECODER1_2: track 0.00 -> 148.5 mm
- net DECODER1_1: track 0.00 -> 146.6 mm
- net DECODER1_3: track 0.00 -> 145.2 mm
- net DECODER1_4: track 0.00 -> 143.5 mm
- net /4_IN3: track 0.00 -> 82.2 mm, vias 0 -> 1
- net /1_IN2: track 0.00 -> 76.8 mm, vias 0 -> 1
- net /4_IN4: track 0.00 -> 76.8 mm, vias 0 -> 1
- net /1_IN1: track 0.00 -> 74.5 mm, vias 0 -> 1
- net /4_IN2: track 0.00 -> 72.0 mm, vias 0 -> 1
- net /4_IN1: track 0.00 -> 71.9 mm, vias 0 -> 1
- net /1_IN4: track 0.00 -> 69.5 mm, vias 0 -> 1
- net /1_IN3: track 0.00 -> 69.2 mm, vias 0 -> 1
- net /3_IN3: track 0.00 -> 66.8 mm, vias 0 -> 1
- net /3_IN4: track 0.00 -> 63.6 mm, vias 0 -> 1
- net /2_IN2: track 0.00 -> 63.4 mm, vias 0 -> 1
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
Commit message: update
Parts:
- moved C43 349.7 mm to (354.3, 279.0)
- moved C44 349.7 mm to (411.6, 267.0)
- moved C7 349.7 mm to (458.1, 273.7)
- moved D1 349.7 mm to (343.1, 281.0)
- moved D17 349.7 mm to (337.6, 281.2)
- moved F1 349.7 mm to (330.2, 279.0)
- moved J2 349.7 mm to (321.1, 284.0)
- moved L1 349.7 mm to (394.8, 280.5)
- moved L2 349.7 mm to (346.6, 279.5)
- moved PS1 349.7 mm to (346.6, 295.5)
- moved C1 349.7 mm to (446.6, 267.2)
- moved D2 349.7 mm to (464.6, 272.8)
- moved R2 349.7 mm to (464.6, 269.0)
- moved U4 349.7 mm to (380.9, 279.5)
- moved U8 349.7 mm to (457.1, 269.0)
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Connections:
- U19 pad 10: Net-(U19-S1) -> /6_IN4
- U19 pad 11: Net-(U19-S0) -> /6_IN3
- U19 pad 12: GND -> unconnected-(U19-VSS-Pad12)
- U19 pad 13: Net-(U19-S13) -> /7_IN2
- U19 pad 14: Net-(U19-S12) -> /7_IN1
- U19 pad 15: Net-(U19-S15) -> /7_IN4
- U19 pad 16: Net-(U19-S14) -> /7_IN3
- U19 pad 17: Net-(U19-S9) -> /8_IN2
- U19 pad 18: Net-(U19-S8) -> /8_IN1
- U19 pad 19: Net-(U19-S11) -> /8_IN4
- U19 pad 20: Net-(U19-S10) -> /8_IN3
- U19 pad 4: Net-(U19-S7) -> /5_IN2
- U19 pad 5: Net-(U19-S6) -> /5_IN1
- U19 pad 6: Net-(U19-S5) -> /5_IN4
- U19 pad 7: Net-(U19-S4) -> /5_IN3
- U19 pad 8: Net-(U19-S3) -> /6_IN2
- U19 pad 9: Net-(U19-S2) -> /6_IN1
- U20 pad 14: Net-(U19-S9) -> /7_IN2
- U20 pad 15: Net-(U19-S8) -> /7_IN1
- U20 pad 6: Net-(U19-S11) -> /7_IN4
- U20 pad 7: Net-(U19-S10) -> /7_IN3
- U21 pad 14: Net-(U19-S13) -> /8_IN2
- U21 pad 15: Net-(U19-S12) -> /8_IN1
- U21 pad 6: Net-(U19-S15) -> /8_IN4
- U21 pad 7: Net-(U19-S14) -> /8_IN3
- U22 pad 14: Net-(U19-S1) -> /5_IN2
- U22 pad 15: Net-(U19-S0) -> /5_IN1
- U22 pad 6: Net-(U19-S3) -> /5_IN4
- U22 pad 7: Net-(U19-S2) -> /5_IN3
- U23 pad 14: Net-(U19-S5) -> /6_IN2
- U23 pad 15: Net-(U19-S4) -> /6_IN1
- U23 pad 6: Net-(U19-S7) -> /6_IN4
- U23 pad 7: Net-(U19-S6) -> /6_IN3
Routing:
- net DE/RE: track 0.00 -> 717.2 mm
- net +5V: track 42.8 -> 615.9 mm, vias 0 -> 2
- net GND: track 177.8 -> 542.8 mm, vias 0 -> 4
- net SPI3_SCK: track 0.00 -> 314.1 mm
- net SPI3_MOSI: track 0.00 -> 305.1 mm
- net +3.3V: track 16.1 -> 297.2 mm, vias 0 -> 3
- net SP3_MISO: track 0.00 -> 234.6 mm
- net DRDY: track 0.00 -> 225.1 mm
- net CS: track 0.00 -> 216.7 mm
- net Net-(U28-S4): track 15.9 -> 223.8 mm
- net UART RX: track 0.00 -> 185.9 mm
- net Net-(U28-S3): track 17.2 -> 202.9 mm
- net UART TX: track 0.00 -> 180.4 mm
- net DECODER2_3: track 0.00 -> 168.7 mm
- net DECODER2_4: track 0.00 -> 165.9 mm
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
Commit message: đã xong các dây dữ liệu
Parts:
- moved SW1 130.6 mm to (738.4, 364.4), turned to 180 degrees
- moved R24 30.3 mm to (596.8, 280.2)
- moved R12 23.9 mm to (749.0, 460.5)
- moved R10 23.1 mm to (749.0, 459.5)
- moved R9 23.0 mm to (749.0, 458.5)
- moved R8 22.9 mm to (749.0, 457.5)
- moved R4 22.8 mm to (749.0, 453.5)
- moved R7 22.8 mm to (749.0, 456.5)
- moved R5 22.8 mm to (749.0, 454.5)
- moved R6 22.7 mm to (749.0, 455.5)
- moved C27 18.4 mm to (750.5, 460.0)
- moved C26 18.2 mm to (750.5, 458.0)
- moved C25 17.8 mm to (750.5, 456.0)
- moved C24 17.8 mm to (750.5, 454.0)
- moved R15 17.2 mm to (756.0, 462.0), turned to -90 degrees
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Connections:
- net SP3_MISO renamed SPI3_MISO
- U2 pad 46: unconnected-(U2-PE15-Pad46) -> DE/RE
- U2 pad 47: unconnected-(U2-PB10-Pad47) -> UART TX
- U2 pad 48: unconnected-(U2-PB11-Pad48) -> UART RX
- U2 pad 68: UART TX -> unconnected-(U2-PA9-Pad68)
- U2 pad 69: UART RX -> unconnected-(U2-PA10-Pad69)
- U2 pad 76: DE/RE -> unconnected-(U2-PA14-Pad76)
Routing:
- net DE/RE: track 717.2 -> 174.5 mm
- net ADC_RESET: track 1.98 -> 202.5 mm
- net SPI3_SCK: track 314.1 -> 201.4 mm
- net SPI3_MOSI: track 305.1 -> 197.1 mm
- net /SW_BOOTO: track 0.00 -> 103.4 mm
- net SPI3_MISO: track 234.6 -> 208.6 mm
- net /AIN7: track 31.4 -> 5.63 mm
- net /AIN6: track 30.7 -> 5.48 mm
- net ADC8: track 557.0 -> 581.6 mm
- net ADC7: track 487.9 -> 512.4 mm
- net /AIN4: track 29.3 -> 5.19 mm
- net ADC6: track 447.9 -> 472.0 mm
- net /AIN5: track 29.4 -> 5.33 mm
- net ADC5: track 415.0 -> 438.7 mm
- net ADC1: track 509.5 -> 533.0 mm
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
Commit message: update
Parts:
- removed C11: 22uF, Capacitor_SMD:C_0805_2012Metric
- added C4: 47uF, Capacitor_THT:C_Radial_D8.0mm_H7.0mm_P3.50mm, F.Cu at (568.8, 286.2)
- C2, C3: value 100nF -> 47uF; footprint Capacitor_SMD:C_0402_1005Metric -> Capacitor_THT:C_Radial_D8.0mm_H7.0mm_P3.50mm
- moved C30 113.8 mm to (724.2, 371.8)
- moved R23 108.2 mm to (721.2, 371.8), turned to 180 degrees
- moved C16 29.9 mm to (601.8, 459.5), turned to -90 degrees
- moved C36 21.1 mm to (620.2, 448.0)
- moved C32 18.8 mm to (620.2, 449.0)
- moved C29 17.3 mm to (619.8, 457.2), turned to -90 degrees
- moved C37 17.0 mm to (618.2, 445.2), turned to 180 degrees
- moved SW1 16.5 mm to (722.5, 368.7)
- moved FB1 15.7 mm to (619.2, 446.5), turned to 180 degrees
- moved C15 14.9 mm to (619.8, 455.2), turned to 90 degrees
- moved C28 13.8 mm to (619.8, 450.5), turned to -90 degrees
- moved C14 12.4 mm to (616.0, 444.8), turned to 180 degrees
- moved C3 9.41 mm to (356.0, 289.5)
- moved C42 7.04 mm to (623.8, 458.8)
- moved C10 5.01 mm to (574.2, 284.3)
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Connections:
- U2 pad 35: CS -> unconnected-(U2-PB0-Pad35)
- U2 pad 36: DRDY -> unconnected-(U2-PB1-Pad36)
- U2 pad 37: ADC_RESET -> unconnected-(U2-PB2-Pad37)
- U2 pad 86: unconnected-(U2-PD5-Pad86) -> ADC_RESET
- U2 pad 87: unconnected-(U2-PD6-Pad87) -> CS
- U2 pad 88: unconnected-(U2-PD7-Pad88) -> DRDY
- Y2 pad 2: unconnected-(Y2-GND-Pad2) -> GND
- Y2 pad 4: unconnected-(Y2-GND-Pad2)_1 -> GND
Routing:
- net Net-(U2-BOOT0): track 0.00 -> 146.9 mm, vias 0 -> 2
- net Net-(U2-NRST): track 0.00 -> 119.5 mm
- net /SW_BOOTO: track 103.4 -> 1.60 mm
- net +3.3V: track 299.1 -> 378.7 mm, vias 3 -> 8
- net GND: track 542.7 -> 592.1 mm, vias 4 -> 8
- net -12V: track 109.6 -> 119.2 mm
- net Net-(U2-PH1): track 5.08 -> 11.6 mm
- net ADC_RESET: track 202.5 -> 208.2 mm
- net CS: track 196.9 -> 202.3 mm
- net DRDY: track 204.7 -> 209.6 mm
- net +3.3VA: track 0.00 -> 3.89 mm
- net +5V_ISO: track 15.9 -> 17.2 mm
- net +12V: track 156.8 -> 158.1 mm
- net GND_ISO: track 66.6 -> 67.4 mm
- net Net-(U2-PH0): track 9.44 -> 10.1 mm
