File: ADC.kicad_pcb (KiCad board)
At the start: 2 copper layers, 195 parts, among them J1 Conn_01x03_Pin, J2 Screw_Terminal_01x02, J3 Screw_Terminal_01x09, SW1 SW_SPDT, U1 ADS1256IDBR, U10 CD4514BM, U11 ADG5412FBCPZ-RL7, U12 ADR421ARMZ, U13 OPA211ID, U14 ADG5412FBCPZ-RL7, U15 OPA211ID, U16 ADG5412FBCPZ-RL7, U17 OPA211ID, U18 CD4072BM, U19 CD4514BM, U2 MCU-STM32F407VET6_LQFP100_, U20 ADG5412FBCPZ-RL7, U21 ADG5412FBCPZ-RL7, U22 ADG5412FBCPZ-RL7, U23 ADG5412FBCPZ-RL7, U24 OPA211ID, U25 OPA211ID, U26 OPA211ID, U27 OPA211ID, U28 CD4043BPWR, U29 TLV1704AIPWR, U3 ADM2483xRW, U30 TLV1704AIPWR, U31 TLV1704AIPWR, U32 CD4072BM, U4 LM2596S-5, U5 DCP010505BP, U6 TLV1704AIPWR, U7 OPA211ID, U8 AMS1117-3.3, U9 ADG5412FBCPZ-RL7, Y1 8MHz, Y2 ABM3B-25.000MHZ-D2Y-T

Commit message: gần như xong
Parts:
- R75, R76, R77, R78: moved to B.Cu
- moved J3 301.9 mm to (548.0, 447.9)
- moved D15 296.4 mm to (557.9, 484.1)
- moved D7 296.0 mm to (557.9, 476.9)
- moved D8 296.0 mm to (557.9, 469.8)
- moved D9 295.7 mm to (557.9, 462.6)
- moved D10 295.7 mm to (557.9, 455.4)
- moved D11 295.4 mm to (557.9, 448.2)
- moved D12 295.4 mm to (557.9, 441.1), turned to -90 degrees
- moved D13 295.2 mm to (557.9, 434.0), turned to 90 degrees
- moved D14 287.8 mm to (553.8, 480.9)
- moved D19 287.4 mm to (553.7, 466.5)
- moved D21 287.1 mm to (553.7, 452.2)
- moved D23 286.9 mm to (553.7, 437.9)
- moved J2 262.1 mm to (547.6, 415.8)
- moved F1 257.9 mm to (551.8, 410.9), turned to 90 degrees
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Connections:
- U10 pad 10: /2_IN4 -> /2_in3
- U10 pad 11: /2_in3 -> /3_IN1
- U10 pad 13: /3_IN2 -> /4_IN3
- U10 pad 14: /3_IN1 -> /4_IN4
- U10 pad 15: /3_IN4 -> /4_IN1
- U10 pad 16: /3_IN3 -> /4_IN2
- U10 pad 17: /4_IN2 -> /3_IN3
- U10 pad 18: /4_IN1 -> /3_IN4
- U10 pad 19: /4_IN4 -> /3_IN2
- U10 pad 20: /4_IN3 -> /2_IN4
- U19 pad 12: unconnected-(U19-VSS-Pad12) -> GND
Routing:
- net +5V: track 615.9 -> 27.4 mm, vias 2 -> 1
- net ADC8: track 581.6 -> 118.9 mm
- net ADC7: track 512.4 -> 109.5 mm
- net ADC6: track 472.0 -> 113.6 mm
- net ADC1: track 533.0 -> 191.2 mm
- net ADC4: track 434.6 -> 99.0 mm
- net ADC2: track 485.4 -> 152.2 mm
- net ADC5: track 438.7 -> 110.9 mm
- net ADC3: track 450.2 -> 126.1 mm
- net -12V: track 119.2 -> 308.7 mm, vias 2 -> 30
- net +12V: track 158.1 -> 338.8 mm, vias 10 -> 26
- net SPI3_SCK: track 201.4 -> 23.1 mm
- net VinP1: track 214.3 -> 38.9 mm
- net CS: track 202.3 -> 28.5 mm
- net DRDY: track 209.6 -> 35.8 mm
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
Commit message: 0k
Parts:
- added H1: MountingHole, MountingHole:MountingHole_2.1mm, F.Cu at (644.0, 423.4)
- added H2: MountingHole, MountingHole:MountingHole_2.1mm, F.Cu at (646.1, 490.1)
- added H3: MountingHole, MountingHole:MountingHole_2.1mm, F.Cu at (548.7, 490.2)
- added H4: MountingHole, MountingHole:MountingHole_2.1mm, F.Cu at (548.7, 421.7)
- C7, D1, D17, D2, D3, F1, L1, L2, R2, U4, U8: moved to F.Cu
- moved J2 100.1 mm to (643.9, 443.2)
- moved F1 88.3 mm to (636.1, 437.1), turned to -90 degrees
- moved D17 84.3 mm to (634.9, 444.9)
- moved D1 75.5 mm to (629.6, 443.1)
- moved L2 72.3 mm to (632.6, 439.2), turned to 180 degrees
- moved C43 58.1 mm to (624.8, 435.4)
- moved U4 33.2 mm to (611.4, 433.4), turned to 0 degrees
- moved U8 31.0 mm to (617.4, 452.9), turned to -90 degrees
- moved R2 30.3 mm to (621.6, 456.3), turned to 90 degrees
- moved D2 27.9 mm to (622.0, 453.7), turned to -90 degrees
- moved C1 25.8 mm to (615.7, 444.2), turned to 0 degrees
- moved C7 25.8 mm to (622.0, 450.4), turned to 90 degrees
- moved R22 23.9 mm to (626.8, 461.7)
- moved J1 23.7 mm to (647.4, 463.5)
- moved D6 23.2 mm to (642.3, 463.6)
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Routing:
- net GND: track 614.6 -> 847.6 mm, vias 28 -> 31
- net +3.3V: track 364.1 -> 474.0 mm, vias 13 -> 19
- net +5V: track 27.4 -> 106.4 mm
- net Net-(PS1-+VIN): track 42.8 -> 81.4 mm
- net -12V: track 308.7 -> 284.0 mm
- net GND_ISO: track 91.3 -> 74.5 mm
- net +5V_ISO: track 43.8 -> 28.6 mm
- net UART RX: track 1.02 -> 12.7 mm
- net Net-(U1-AVDD): track 5.30 -> 16.5 mm, vias 0 -> 2
- net DE/RE: track 5.40 -> 11.4 mm
- net Net-(U3-B): track 10.5 -> 15.1 mm
- net UART TX: track 1.02 -> 5.51 mm
- net +12V_IN: track 5.11 -> 9.07 mm
- net Net-(D1-K): track 16.4 -> 13.9 mm
- net Net-(U2-NRST): track 27.1 -> 29.6 mm
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- added copper zone on B.Cu, net GND

Commit message: update
Parts:
- moved C34 0.17 mm to (633.0, 474.1)
- moved C35 0.12 mm to (631.8, 474.4)
Changed lines of the file:
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@@
 		(tags "C Radial series Radial pin pitch 3.50mm diameter 8mm height 7mm Non-Polar Electrolytic Capacitor")
 		(property "Reference" "C4"
-			(at 1.75 -5.25 360)
+			(at 1.75 -5.25 0)
 			(layer "F.SilkS")
 			(effects
@@
 		)
 		(property "Value" "47uF"
-			(at 1.75 5.25 360)
+			(at 1.75 5.25 0)
 			(layer "F.Fab")
 			(effects
@@
 		)
 		(fp_text user "${REFERENCE}"
-			(at 1.75 0 360)
+			(at 1.75 0 0)
 			(layer "F.Fab")
 			(effects
@@
 		)
 		(fp_text user "${REFERENCE}"
-			(at 0 0 360)
+			(at 0 0 0)
 			(layer "F.Fab")
 			(effects
@@
 		(tags "C Radial series Radial pin pitch 3.50mm diameter 8mm height 7mm Non-Polar Electrolytic Capacitor")
 		(property "Reference" "C1"
-			(at 1.75 -5.25 360)
+			(at 1.75 -5.25 0)
 			(layer "F.SilkS")
 			(effects
@@
 		)
 		(property "Value" "47uF"
-			(at 1.75 5.25 360)
+			(at 1.75 5.25 0)
 			(layer "F.Fab")
 			(effects
@@
 		)
 		(fp_text user "${REFERENCE}"
-			(at 1.75 0 360)
+			(at 1.75 0 0)
 			(layer "F.Fab")
 			(effects
@@
 	(footprint "Capacitor_SMD:C_0402_1005Metric"
 		(layer "F.Cu")
-		(at 632.959137 474.220735 -90)
+		(at 633.05 474.08 -90)
 		(descr "Capacitor SMD 0402 (1005 Metric), square (rectangular) end terminal, IPC_7351 nominal, (Body size source: IPC-SM-782 page 76, https://www.pcb-3d.com/wordpress/wp-content/uploads/ipc-sm-782a_amendment_1_and_2.pdf), generated with kicad-footprint-generator")
 		(tags "capacitor")
@@
 		(at 596.075 439.91 180)
 		(property "Reference" "U5"
-			(at -3.30232 -19.4583 360)
+			(at -3.30232 -19.4583 0)
 			(layer "F.SilkS")
 			(effects
@@
 		)
 		(property "Value" "DCP010505BP"
-			(at 10.445985 4.041125 360)
+			(at 10.445985 4.041125 0)
 			(layer "F.Fab")
 			(effects
@@
 		)
 		(property "Footprint" "DCP10505BP:DIP254P762X533-7P"
-			(at 0 0 360)
+			(at 0 0 0)
 			(layer "F.Fab")
 			(hide yes)
@@
 		)
 		(property "Datasheet" ""
-			(at 0 0 360)
+			(at 0 0 0)
 			(layer "F.Fab")
 			(hide yes)
@@
 		)
 		(property "Description" ""
-			(at 0 0 360)
+			(at 0 0 0)
 			(layer "F.Fab")
 			(hide yes)
@@
 	(footprint "Capacitor_SMD:C_0603_1608Metric"
 		(layer "F.Cu")
-		(at 631.916637 474.358235 -90)
+		(at 631.8 474.375 -90)
 		(descr "Capacitor SMD 0603 (1608 Metric), square (rectangular) end terminal, IPC_7351 nominal, (Body size source: IPC-SM-782 page 76, https://www.pcb-3d.com/wordpress/wp-content/uploads/ipc-sm-782a_amendment_1_and_2.pdf), generated with kicad-footprint-generator")
 		(tags "capacitor")
@@
 	(via
 		(at 631.075 473.695735)
-		(size 0.6)
-		(drill 0.3)
+		(size 0.2)
+		(drill 0.2)
 		(layers "F.Cu" "B.Cu")
 		(net 25)
